Commit message: make obstacles lighter

File: push_policy/resources/obstacle1.urdf (robot description, URDF)
Before this commit: robot obstacle1, 1 links, 0 joints
Links:
- link base_link: mass 2 -> 1

File: push_policy/resources/obstacle2.urdf (robot description, URDF)
Before this commit: robot obstacle2, 1 links, 0 joints
Links:
- link base_link: mass 3 -> 1.5

File: push_policy/resources/obstacle3.urdf (robot description, URDF)
Before this commit: robot obstacle3, 1 links, 0 joints
Links:
- link base_link: mass 4 -> 2

File: push_policy/resources/obstacle4.urdf (robot description, URDF)
Before this commit: robot obstacle2, 1 links, 0 joints
Links:
- link base_link: mass 100 -> 50

File: push_policy/resources/obstacle5.urdf (robot description, URDF)
Before this commit: robot obstacle3, 1 links, 0 joints
Links:
- link base_link: mass 4.5 -> 2.25
