Commit message: add head link

File: push_policy/resources/car.urdf (robot description, URDF)
Before this commit: robot simplecar, 7 links, 6 joints
Links:
- added link head; collision box size=0.1 0.3 0.1; visual box size=0.1 0.3 0.1
Joints:
- added joint base_to_head: type fixed, parent base_link, child head, origin xyz=0.3 0 0

Commit message: add head inertia

File: push_policy/resources/car.urdf (robot description, URDF)
Before this commit: robot simplecar, 8 links, 7 joints
Links:
- link head: mass None -> 2
