Commit message: tweak urdfs

File: push_policy/resources/obstacle4.urdf (robot description, URDF)
Before this commit: robot obstacle2, 1 links, 0 joints
Links:
- link base_link: mass 50 -> 5

File: push_policy/resources/obstacle5.urdf (robot description, URDF)
Before this commit: robot obstacle3, 1 links, 0 joints
Links:
- link base_link: geometry collision cylinder length=0.4 radius=0.4; visual cylinder length=0.1 radius=0.4
